Commit message: add book

File: chatp6/chapt6_ws/src/fishbot_description/urdf/fishbot/action/caster.urdf.xacro (robot description, xacro)
@@ -24,4 +24,13 @@
                 </material>
             </visual>
+            <collision>
+                <origin xyz="0.0 0.0 0.0" rpy="0.0 0.0 0.0"/>
+                <geometry>
+                    <sphere radius="0.016"/>
+                </geometry>
+                <material name="yellow">
+                    <color rgba="1.0 1.0 0.0 0.8"/>
+                </material>
+            </collision>
         </link>
         <!-- 定义 caster 与 base_link 的固定 joint -->

File: chatp6/chapt6_ws/src/fishbot_description/urdf/fishbot/action/wheel.urdf.xacro (robot description, xacro)
@@ -24,4 +24,13 @@
                 </material>
             </visual>
+            <collision>
+                <origin xyz="0.0 0.0 0.0" rpy="1.57097 0.0 0.0"/>
+                <geometry>
+                    <cylinder radius="0.032" length="0.04"/>
+                </geometry>
+                <material name="yellow">
+                    <color rgba="1.0 1.0 0.0 0.8"/>
+                </material>
+            </collision>
         </link>
         <!-- 定义 wheel 与 base_link 的固定 joint -->

File: chatp6/chapt6_ws/src/fishbot_description/urdf/fishbot/base.urdf.xacro (robot description, xacro)
@@ -17,4 +17,5 @@
     -->
     <xacro:macro name="base_xacro" params="base_length base_radius">
+        <link name="robot_footprint" />
         <!-- 定义底盘 link -->
         <link name="base_link">
@@ -28,5 +29,19 @@
                 </material>
             </visual>
+            <collision>
+                <origin xyz="0.0 0.0 0.0" rpy="0.0 0.0 0.0"/>
+                <geometry>
+                    <cylinder radius="${base_radius}" length="${base_length}"/>
+                </geometry>
+                <material name="white">
+                    <color rgba="${color_white}"/>
+                </material>
+            </collision>
         </link>
+        <joint name="footprint_joint" type="fixed">
+            <origin xyz="0.0 0.0 ${base_length/2.0+0.032}" rpy="0.0 0.0 0.0"/>
+            <parent link="robot_footprint"/>
+            <child link="base_link"/>
+        </joint>
     </xacro:macro>
 </robot>

File: chatp6/chapt6_ws/src/fishbot_description/urdf/fishbot/firstbot.urdf.xacro (robot description, xacro)
@@ -16,5 +16,5 @@
     <xacro:wheel_xacro wheel_name="left_wheel" xyz="0 0.1 -0.06" />
     <xacro:wheel_xacro wheel_name="right_wheel" xyz="0 -0.1 -0.06" />
-    <xacro:caster_xacro caster_name="front_caster" xyz="0.08 0.0 -0.06" />
-    <xacro:caster_xacro caster_name="back_caster" xyz="-0.08 0.0 -0.06" />
+    <xacro:caster_xacro caster_name="front_caster" xyz="0.08 0.0 -0.076" />
+    <xacro:caster_xacro caster_name="back_caster" xyz="-0.08 0.0 -0.076" />
 </robot>

File: chatp6/chapt6_ws/src/fishbot_description/urdf/fishbot/sensor/camera.urdf.xacro (robot description, xacro)
@@ -30,4 +30,13 @@
                 </material>
             </visual>
+            <collision>
+                <origin xyz="0.0 0.0 0.0" rpy="0.0 0.0 0.0"/>
+                <geometry>
+                    <box size="${imu_size} ${imu_size} ${imu_size}"/>
+                </geometry>
+                <material name="green">
+                    <color rgba="${color_green}"/>
+                </material>
+            </collision>
         </link>
         <!-- 定义摄像头与 base_link 的固定 joint -->

File: chatp6/chapt6_ws/src/fishbot_description/urdf/fishbot/sensor/imu.urdf.xacro (robot description, xacro)
@@ -28,4 +28,13 @@
                 </material>
             </visual>
+            <collision>
+                <origin xyz="0.0 0.0 0.0" rpy="0.0 0.0 0.0"/>
+                <geometry>
+                    <box size="${imu_size} ${imu_size} ${imu_size}"/>
+                </geometry>
+                <material name="black">
+                    <color rgba="${color_black}"/>
+                </material>
+            </collision>
         </link>
         <!-- 定义 IMU 与 base_link 的固定 joint -->

File: chatp6/chapt6_ws/src/fishbot_description/urdf/fishbot/sensor/laser.urdf.xacro (robot description, xacro)
@@ -5,24 +5,34 @@
     作者：hzy
     日期：2025-07-11
+    描述：
+        1. 支撑杆（绿色）和雷达主体（红色）均包含可视化与碰撞体属性。
+        2. 支撑杆通过 joint 连接到底盘 base_link，雷达主体通过 joint 连接支撑杆。
+        3. 所有参数均可灵活调整，便于模型扩展。
 -->
 <robot name="fishbot" xmlns:xacro="http://ros.org/wiki/xacro">
-    <!-- 激光传感器支撑杆尺寸参数 -->
+    <!-- 支撑杆尺寸参数（绿色），用于定义支撑杆的半径和长度 -->
     <xacro:property name="laser_cy_radius" value="0.005"/>
     <xacro:property name="laser_cy_length" value="0.05" />
-    <!-- 雷达参数 -->
+    <!-- 雷达主体参数（红色），用于定义雷达的半径和长度 -->
     <xacro:property name="laser_radius" value="0.02" />
     <xacro:property name="laser_length" value="0.02" />
-    <!-- 激光传感器颜色参数 -->
+    <!-- 颜色参数，分别用于支撑杆（绿色）、雷达主体（红色）、备用黑色 -->
     <xacro:property name="color_green" value="0.0 1.0 0.0 0.8"/>
     <xacro:property name="color_black" value="0.0 0.0 0.0 0.8"/>
+    <!-- 红色参数，应用于雷达主体 -->
+    <xacro:property name="color_red" value="1.0 0.0 0.0 0.8"/>
     <!--
         宏：laser_xacro
-        参数：imu_size, color_black, xyz
-        功能：生成激光传感器 link 及其与 base_link 的固定 joint
+        参数：xyz（支撑杆在 base_link 下的位置）
+        功能：
+            1. 生成激光传感器支撑杆（绿色）和雷达主体（红色）
+            2. 支撑杆与 base_link 通过 joint 连接
+            3. 雷达主体与支撑杆通过 joint 连接
     -->
     <xacro:macro name="laser_xacro" params="xyz">
-        <!-- 定义激光传感器支撑杆 link -->
+        <!-- 支撑杆 link（绿色），包含可视化和碰撞体 -->
         <link name="laser_cylinder_link">
             <visual>
+                <!-- 支撑杆可视化部分，绿色 -->
                 <origin xyz="0.0 0.0 0.0" rpy="0.0 0.0 0.0"/>
                 <geometry>
@@ -33,19 +43,41 @@
                 </material>
             </visual>
+            <collision>
+                <!-- 支撑杆碰撞体部分，绿色 -->
+                <origin xyz="0.0 0.0 0.0" rpy="0.0 0.0 0.0"/>
+                <geometry>
+                    <cylinder radius="${laser_cy_radius}" length="${laser_cy_length}"/>
+                </geometry>
+                <material name="green">
+                    <color rgba="${color_green}"/>
+                </material>
+            </collision>
         </link>
-        <!-- 雷达 -->
+        <!-- 雷达主体 link（红色），包含可视化和碰撞体 -->
         <link name="laser_link">
             <visual>
+                <!-- 雷达主体可视化部分，红色 -->
                 <origin xyz="0.0 0.0 0.0" rpy="0.0 0.0 0.0"/>
                 <geometry>
                     <cylinder radius="${laser_radius}" length="${laser_length}"/>
                 </geometry>
-                <material name="black">
-                    <color rgba="${color_black}"/>
+                <material name="red">
+                    <color rgba="${color_red}"/>
                 </material>
             </visual>
+            <collision>
+                <!-- 雷达主体碰撞体部分，红色 -->
+                <origin xyz="0.0 0.0 0.0" rpy="0.0 0.0 0.0"/>
+                <geometry>
+                    <cylinder radius="${laser_radius}" length="${laser_length}"/>
+                </geometry>
+                <material name="red">
+                    <color rgba="${color_red}"/>
+                </material>
+            </collision>
         </link>
-        <!-- 定义激光传感器与 base_link 的固定 joint -->
+        <!-- 雷达主体与支撑杆的固定 joint -->
         <joint name="laser_joint" type="fixed">
+            <!-- 雷达主体与支撑杆连接 -->
             <parent link="laser_cylinder_link"/>
             <child link="laser_link"/>
@@ -53,4 +85,5 @@
         </joint>
         <joint name="laser_cylinker_link" type="fixed">
+            <!-- 支撑杆与 base_link 连接 -->
             <parent link="base_link"/>
             <child link="laser_cylinder_link"/>

Commit message: add mess and inertia

File: chatp6/chapt6_ws/src/fishbot_description/urdf/fishbot/action/caster.urdf.xacro (robot description, xacro)
@@ -7,4 +7,5 @@
 -->
 <robot name="fishbot" xmlns:xacro="http://ros.org/wiki/xacro">
+   <xacro:include filename="$(find fishbot_description)/urdf/fishbot/common_inertia.xacro" />
     <!--
         宏：caster_xacro
@@ -33,4 +34,5 @@
                 </material>
             </collision>
+            <xacro:sphere_inertia m="0.01" r="0.016" />
         </link>
         <!-- 定义 caster 与 base_link 的固定 joint -->

File: chatp6/chapt6_ws/src/fishbot_description/urdf/fishbot/action/wheel.urdf.xacro (robot description, xacro)
@@ -7,4 +7,5 @@
 -->
 <robot name="fishbot" xmlns:xacro="http://ros.org/wiki/xacro">
+   <xacro:include filename="$(find fishbot_description)/urdf/fishbot/common_inertia.xacro" />
     <!--
         宏：wheel_xacro
@@ -33,4 +34,5 @@
                 </material>
             </collision>
+            <xacro:cylinder_inertia m="0.1" h="0.04" r="0.032"/>
         </link>
         <!-- 定义 wheel 与 base_link 的固定 joint -->

File: chatp6/chapt6_ws/src/fishbot_description/urdf/fishbot/base.urdf.xacro (robot description, xacro)
@@ -7,4 +7,5 @@
 -->
 <robot name="fishbot" xmlns:xacro="http://ros.org/wiki/xacro">
+    <xacro:include filename="$(find fishbot_description)/urdf/fishbot/common_inertia.xacro" />
     <!-- 底盘参数定义 -->
     <!-- <xacro:property name="base_radius" value="0.10"/>
@@ -38,4 +39,5 @@
                 </material>
             </collision>
+            <xacro:cylinder_inertia m="1.0" r="${base_radius}" h="${base_length}"/>
         </link>
         <joint name="footprint_joint" type="fixed">

File: chatp6/chapt6_ws/src/fishbot_description/urdf/fishbot/firstbot.urdf.xacro (robot description, xacro)
@@ -12,6 +12,6 @@
     <xacro:base_xacro base_radius="0.1" base_length="0.12" />
     <xacro:imu_xacro xyz="0.0 0.0 0.05" />
-    <xacro:camera_xacro xyz="0.09 0 0.07" />
-    <xacro:laser_xacro xyz="0.0 0.0 0.08" />
+    <xacro:camera_xacro xyz="0.09 0.0 0.07" />
+    <xacro:laser_xacro xyz="0.06 0.0 0.07" />
     <xacro:wheel_xacro wheel_name="left_wheel" xyz="0 0.1 -0.06" />
     <xacro:wheel_xacro wheel_name="right_wheel" xyz="0 -0.1 -0.06" />

File: chatp6/chapt6_ws/src/fishbot_description/urdf/fishbot/sensor/camera.urdf.xacro (robot description, xacro)
@@ -7,4 +7,5 @@
 -->
 <robot name="fishbot" xmlns:xacro="http://ros.org/wiki/xacro">
+   <xacro:include filename="$(find fishbot_description)/urdf/fishbot/common_inertia.xacro" />
     <!-- 摄像头相关参数定义 -->
     <xacro:property name="base_radius" value="0.10"/>
@@ -39,4 +40,5 @@
                 </material>
             </collision>
+            <xacro:box_inertia m="0.01" w="0.02" h="0.10" d="0.02" />
         </link>
         <!-- 定义摄像头与 base_link 的固定 joint -->

File: chatp6/chapt6_ws/src/fishbot_description/urdf/fishbot/sensor/imu.urdf.xacro (robot description, xacro)
@@ -7,4 +7,5 @@
 -->
 <robot name="fishbot" xmlns:xacro="http://ros.org/wiki/xacro">
+   <xacro:include filename="$(find fishbot_description)/urdf/fishbot/common_inertia.xacro" />
     <!-- IMU 传感器尺寸参数 -->
     <xacro:property name="imu_size" value="0.02"/>
@@ -37,4 +38,5 @@
                 </material>
             </collision>
+            <xacro:box_inertia m="0.01" w="0.02" d="0.02" h="0.02"/>
         </link>
         <!-- 定义 IMU 与 base_link 的固定 joint -->

File: chatp6/chapt6_ws/src/fishbot_description/urdf/fishbot/sensor/laser.urdf.xacro (robot description, xacro)
@@ -11,4 +11,5 @@
 -->
 <robot name="fishbot" xmlns:xacro="http://ros.org/wiki/xacro">
+    <xacro:include filename="$(find fishbot_description)/urdf/fishbot/common_inertia.xacro" />
     <!-- 支撑杆尺寸参数（绿色），用于定义支撑杆的半径和长度 -->
     <xacro:property name="laser_cy_radius" value="0.005"/>
@@ -53,4 +54,5 @@
                 </material>
             </collision>
+            <xacro:cylinder_inertia m="0.01" r="0.01" h="0.10" />
         </link>
         <!-- 雷达主体 link（红色），包含可视化和碰撞体 -->
@@ -76,18 +78,19 @@
                 </material>
             </collision>
+            <xacro:cylinder_inertia m="0.03" r="0.02" h="0.02" />
         </link>
-        <!-- 雷达主体与支撑杆的固定 joint -->
-        <joint name="laser_joint" type="fixed">
-            <!-- 雷达主体与支撑杆连接 -->
-            <parent link="laser_cylinder_link"/>
-            <child link="laser_link"/>
-            <origin xyz="0.0 0.0 0.035" rpy="0.0 0.0 0.0"/>
-        </joint>
+        <!-- 支撑杆与 base_link 连接  -->
         <joint name="laser_cylinker_link" type="fixed">
-            <!-- 支撑杆与 base_link 连接 -->
             <parent link="base_link"/>
             <child link="laser_cylinder_link"/>
             <origin xyz="${xyz}" rpy="0.0 0.0 0.0"/>
         </joint>
+        <!-- 雷达主体与支撑杆的固定 joint -->
+        <joint name="laser_joint" type="fixed">
+            <!-- 雷达主体与支撑杆连接 -->
+            <parent link="base_link"/>
+            <child link="laser_link"/>
+            <origin xyz="0.06 0.0 0.09" rpy="0.0 0.0 0.0"/>
+        </joint>
     </xacro:macro>
 </robot>

Commit message: 加载 robot 到 world

File: chatp6/chapt6_ws/src/fishbot_description/urdf/fishbot/action/caster.urdf.xacro (robot description, xacro)
@@ -42,4 +42,12 @@
             <origin xyz="${xyz}" rpy="0.0 0.0 0.0"/>
         </joint>
+        <!-- 定义 caster 的 caster_joint -->
+        <gazebo reference="${caster_name}_link">
+            <material>Gazebo/Black</material>
+            <mu1 value="0.0" />
+            <mu2 value="0.0" />
+            <kp value="1000000000.0" />
+            <kd value="1.0" />
+        </gazebo>
     </xacro:macro>
 </robot>

File: chatp6/chapt6_ws/src/fishbot_description/urdf/fishbot/action/wheel.urdf.xacro (robot description, xacro)
@@ -43,4 +43,11 @@
             <axis xyz="0.0 1.0 0.0"/>
         </joint>
+        <gazebo reference="${wheel_name}_link">
+            <material>Gazebo/Black</material>
+            <mu1 value="20.0" />
+            <mu2 value="20.0" />
+            <kp value="1000000000.0" />
+            <kd value="1.0" />
+        </gazebo>
     </xacro:macro>
 </robot>

File: chatp6/chapt6_ws/src/fishbot_description/urdf/fishbot/base.urdf.xacro (robot description, xacro)
@@ -46,4 +46,7 @@
             <child link="base_link"/>
         </joint>
+        <gazebo reference="base_link">
+            <material>Gazebo/White</material>
+        </gazebo>
     </xacro:macro>
 </robot>

File: chatp6/chapt6_ws/src/fishbot_description/urdf/fishbot/sensor/camera.urdf.xacro (robot description, xacro)
@@ -48,4 +48,7 @@
             <origin xyz="${xyz}" rpy="0.0 0.0 0.0"/>
         </joint>
+        <gazebo reference="camera_link">
+            <material>Gazebo/Blue</material>
+        </gazebo>
     </xacro:macro>
 </robot>

File: chatp6/chapt6_ws/src/fishbot_description/urdf/fishbot/sensor/laser.urdf.xacro (robot description, xacro)
@@ -93,4 +93,10 @@
             <origin xyz="0.06 0.0 0.09" rpy="0.0 0.0 0.0"/>
         </joint>
+        <gazebo reference="laser_cylinder_link">
+            <material>Gazebo/Green</material>
+        </gazebo>
+        <gazebo reference="laser_link">
+            <material>Gazebo/Red</material>
+        </gazebo>
     </xacro:macro>
 </robot>
