Commit message: 添加了深度相机扫描

File: chatp6/chapt6_ws/src/fishbot_description/urdf/fishbot/firstbot.urdf.xacro (robot description, xacro)
@@ -13,4 +13,5 @@
     <xacro:include filename="$(find fishbot_description)/urdf/fishbot/plugins/gazebo_control_plugin.xacro" />
     <xacro:include filename="$(find fishbot_description)/urdf/fishbot/plugins/gazebo_sensor_plugin.xacro" />
+    <xacro:include filename="$(find fishbot_description)/urdf/fishbot/fishbot.ros2_control.xacro" />
     <xacro:base_xacro base_radius="0.1" base_length="0.12" />
     <xacro:imu_xacro xyz="0.0 0.0 0.05" />
@@ -21,5 +22,6 @@
     <xacro:caster_xacro caster_name="front_caster" xyz="0.08 0.0 -0.076" />
     <xacro:caster_xacro caster_name="back_caster" xyz="-0.08 0.0 -0.076" />
-    <xacro:gazebo_control_plugin />
+    <!-- <xacro:gazebo_control_plugin /> -->
     <xacro:gazebo_sensor_plugin />
+    <xacro:fishbot_ros2_control />
 </robot>

File: chatp6/chapt6_ws/src/fishbot_description/urdf/fishbot/plugins/gazebo_sensor_plugin.xacro (robot description, xacro)
@@ -114,5 +114,5 @@
     <sensor type="depth" name="camera_sensor">
         <plugin name="depth_camera" filename="libgazebo_ros_camera.so">
-            <frame_name>camera_optical_link</frame_name>
+            <frame_name>camera_optional_link</frame_name>
         </plugin>
         <always_on>true</always_on>

File: chatp6/chapt6_ws/src/fishbot_description/urdf/fishbot/sensor/camera.urdf.xacro (robot description, xacro)
@@ -42,4 +42,5 @@
             <xacro:box_inertia m="0.01" w="0.02" h="0.10" d="0.02" />
         </link>
+        <link name="camera_optional_link"></link>
         <!-- 定义摄像头与 base_link 的固定 joint -->
         <joint name="camera_joint" type="fixed">
@@ -48,4 +49,9 @@
             <origin xyz="${xyz}" rpy="0.0 0.0 0.0"/>
         </joint>
+        <joint name="camera_optional_joint" type="fixed">
+            <parent link="camera_link" />
+            <child link="camera_optional_link" />
+            <origin xyz="0 0 0" rpy="${-pi/2} 0 ${-pi/2}" />
+        </joint>
         <gazebo reference="camera_link">
             <material>Gazebo/Blue</material>
